Commit message: [Update] Current robot condition

File: urdf/robot_covid.xacro (robot description, xacro)
@@ -144,7 +144,3 @@
     <xacro:arg name="add_plug" default="false"/>
     <xacro:arg name="use_mesh" default="false"/>
-    <xacro:include filename="$(find realsense2_description)/urdf/_l515.urdf.xacro"/>
-    <xacro:sensor_l515 parent="base_link" use_nominal_extrinsics="$(arg use_nominal_extrinsics)" add_plug="$(arg add_plug)" use_mesh="$(arg use_mesh)">
-    <origin xyz="0.1 0.0 ${robot_height + 0.03}" rpy="0.0 0.0 0.0"/>
-    </xacro:sensor_l515>
 </robot>
